File: keeb.kicad_pcb (KiCad board)
At the start: 2 copper layers, 189 parts, among them SW1 SW_Push, U1 ATmega32U4-A, Y1 16MHz

Commit message: arcade session 5
moving stuff
Parts:
- added MX31: tab, PCM_marbastlib-mx:SW_MX_HS_CPG151101S11_1u, F.Cu at (308.1, 77.9)
- moved MX15 507.5 mm to (311.1, 33.3)
- moved MX30 494.6 mm to (311.1, 57.1)
- moved MX14 487.6 mm to (292.1, 33.3)
- moved MX11 469.5 mm to (234.9, 33.3)
- moved MX13 468.1 mm to (273.1, 33.3)
- moved MX29 464.2 mm to (282.6, 57.1)
- moved MX44 451.9 mm to (279.9, 76.2)
- moved MX12 449.0 mm to (254.0, 33.3)
- moved MX10 446.9 mm to (215.9, 33.3)
- moved MX28 434.1 mm to (254.0, 57.1)
- moved MX43 430.1 mm to (260.9, 76.2)
- moved MX9 424.4 mm to (196.8, 33.3)
- moved MX27 413.8 mm to (234.9, 57.1)
- moved MX42 408.6 mm to (241.8, 76.2)
- moved MX8 402.1 mm to (177.8, 33.3)
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
Commit message: fixed mistakes
Parts:
- removed the MX31 at (308.1, 77.9)
- removed S1: MX_stab, PCM_marbastlib-mx:STAB_MX_P_6.25u
- removed S2, S4: MX_stab, PCM_marbastlib-mx:STAB_MX_2u
- removed S3: MX_stab, PCM_marbastlib-mx:STAB_MX_P_2u
- added C8: 0.1uF, Capacitor_SMD:C_0805_2012Metric, B.Cu at (100.8, 136.5)
- C1, C2, C3, C4, C5, C6, C7, D1, D10, D11, D12, D13, D14, D15, D16, D17, D18, D19, D2, D20, D21, D22, D23, D24, D25, D26, D27, D28, D29, D3, D30, D31, D32, D33, D34, D35, D36, D37, D38, D39, D4, D40, D41, D42, D43, D44, D45, D46, D47, D48, D49, D5, D50, D51, D52, D53, D54, D55, D56, D57, D58, D59, D6, D60, D61, D62, D63, D64, D65, D66, D67, D68, D69, D7, D70, D71, D72, D73, D74, D75, D76, D77, D78, D79, D8, D80, D81, D82, D83, D84, D9, F1, R1, R2, R3, R4, R5, R6, SW1, USB1, Y1: moved to B.Cu
- MX1: value Esc -> esc; footprint PCM_marbastlib-mx:SW_MX_HS_CPG151101S11_1u -> MX_Alps_Hybrid:MX-Alps-Hybrid-1U
- MX10: value F9 -> f9; footprint PCM_marbastlib-mx:SW_MX_HS_CPG151101S11_1u -> MX_Alps_Hybrid:MX-Alps-Hybrid-1U
- MX11: value F10 -> f10; footprint PCM_marbastlib-mx:SW_MX_HS_CPG151101S11_1u -> MX_Alps_Hybrid:MX-Alps-Hybrid-1U
- MX12: value F11 -> f11; footprint PCM_marbastlib-mx:SW_MX_HS_CPG151101S11_1u -> MX_Alps_Hybrid:MX-Alps-Hybrid-1U
- MX13: value F12 -> f12; footprint PCM_marbastlib-mx:SW_MX_HS_CPG151101S11_1u -> MX_Alps_Hybrid:MX-Alps-Hybrid-1U
- MX14: value PrtSc -> prtsc; footprint PCM_marbastlib-mx:SW_MX_HS_CPG151101S11_1u -> MX_Alps_Hybrid:MX-Alps-Hybrid-1U
- MX15: value Delete -> del; footprint PCM_marbastlib-mx:SW_MX_HS_CPG151101S11_1u -> MX_Alps_Hybrid:MX-Alps-Hybrid-1U
- MX16, MX17, MX18, MX19, MX20, MX21, MX22, MX23, MX24, MX25, MX26, MX27, MX32, MX33, MX34, MX35, MX36, MX37, MX38, MX39, MX40, MX41, MX47, MX48, MX49, MX50, MX51, MX52, MX53, MX54, MX55, MX59, MX61, MX62, MX63, MX64, MX65, MX66, MX67, MX72, MX73, MX78, MX79, MX80, MX81, MX83: footprint PCM_marbastlib-mx:SW_MX_HS_CPG151101S11_1u -> MX_Alps_Hybrid:MX-Alps-Hybrid-1U
- MX2: value F1 -> f1; footprint PCM_marbastlib-mx:SW_MX_HS_CPG151101S11_1u -> MX_Alps_Hybrid:MX-Alps-Hybrid-1U
- MX28: value + -> =; footprint PCM_marbastlib-mx:SW_MX_HS_CPG151101S11_1u -> MX_Alps_Hybrid:MX-Alps-Hybrid-1U
- MX29: footprint PCM_marbastlib-mx:SW_MX_HS_CPG151101S11_1u -> MX_Alps_Hybrid:MX-Alps-Hybrid-2U-ReversedStabilizers
- MX3: value F2 -> f2; footprint PCM_marbastlib-mx:SW_MX_HS_CPG151101S11_1u -> MX_Alps_Hybrid:MX-Alps-Hybrid-1U
- MX30: value pgUp -> pgup; footprint PCM_marbastlib-mx:SW_MX_HS_CPG151101S11_1u -> MX_Alps_Hybrid:MX-Alps-Hybrid-1U
- MX31: footprint PCM_marbastlib-mx:SW_MX_HS_CPG151101S11_1u -> MX_Alps_Hybrid:MX-Alps-Hybrid-1.5U
- MX4: value F3 -> f3; footprint PCM_marbastlib-mx:SW_MX_HS_CPG151101S11_1u -> MX_Alps_Hybrid:MX-Alps-Hybrid-1U
- MX42: value { -> [; footprint PCM_marbastlib-mx:SW_MX_HS_CPG151101S11_1u -> MX_Alps_Hybrid:MX-Alps-Hybrid-1U
- MX43: value } -> ]; footprint PCM_marbastlib-mx:SW_MX_HS_CPG151101S11_1u -> MX_Alps_Hybrid:MX-Alps-Hybrid-1U
- MX44: value | -> \; footprint PCM_marbastlib-mx:SW_MX_HS_CPG151101S11_1u -> MX_Alps_Hybrid:MX-Alps-Hybrid-1.5U
- MX45: value pgDn -> pgdn; footprint PCM_marbastlib-mx:SW_MX_HS_CPG151101S11_1u -> MX_Alps_Hybrid:MX-Alps-Hybrid-1U
- MX46, MX71: footprint PCM_marbastlib-mx:SW_MX_HS_CPG151101S11_1u -> MX_Alps_Hybrid:MX-Alps-Hybrid-1.75U
- MX5: value F4 -> f4; footprint PCM_marbastlib-mx:SW_MX_HS_CPG151101S11_1u -> MX_Alps_Hybrid:MX-Alps-Hybrid-1U
- MX56: value : -> ;; footprint PCM_marbastlib-mx:SW_MX_HS_CPG151101S11_1u -> MX_Alps_Hybrid:MX-Alps-Hybrid-1U
- MX57: value " -> '; footprint PCM_marbastlib-mx:SW_MX_HS_CPG151101S11_1u -> MX_Alps_Hybrid:MX-Alps-Hybrid-1U
- MX58, MX60: footprint PCM_marbastlib-mx:SW_MX_HS_CPG151101S11_1u -> MX_Alps_Hybrid:MX-Alps-Hybrid-2.25U-ReversedStabilizers
- MX6: value F5 -> f5; footprint PCM_marbastlib-mx:SW_MX_HS_CPG151101S11_1u -> MX_Alps_Hybrid:MX-Alps-Hybrid-1U
- MX68: value < -> ,; footprint PCM_marbastlib-mx:SW_MX_HS_CPG151101S11_1u -> MX_Alps_Hybrid:MX-Alps-Hybrid-1U
- MX69: value > -> .; footprint PCM_marbastlib-mx:SW_MX_HS_CPG151101S11_1u -> MX_Alps_Hybrid:MX-Alps-Hybrid-1U
- MX7: value F6 -> f6; footprint PCM_marbastlib-mx:SW_MX_HS_CPG151101S11_1u -> MX_Alps_Hybrid:MX-Alps-Hybrid-1U
- MX70: value ? -> /; footprint PCM_marbastlib-mx:SW_MX_HS_CPG151101S11_1u -> MX_Alps_Hybrid:MX-Alps-Hybrid-1U
- MX74, MX75, MX76: footprint PCM_marbastlib-mx:SW_MX_HS_CPG151101S11_1u -> MX_Alps_Hybrid:MX-Alps-Hybrid-1.25U
- MX77: footprint PCM_marbastlib-mx:SW_MX_HS_CPG151101S11_1u -> MX_Alps_Hybrid:MX-Alps-Hybrid-6.25U-ReversedStabilizers
- MX8: value F7 -> f7; footprint PCM_marbastlib-mx:SW_MX_HS_CPG151101S11_1u -> MX_Alps_Hybrid:MX-Alps-Hybrid-1U
- MX82: value down -> bottom; footprint PCM_marbastlib-mx:SW_MX_HS_CPG151101S11_1u -> MX_Alps_Hybrid:MX-Alps-Hybrid-1U
- MX9: value F8 -> f8; footprint PCM_marbastlib-mx:SW_MX_HS_CPG151101S11_1u -> MX_Alps_Hybrid:MX-Alps-Hybrid-1U
- moved MX45 457.4 mm to (311.1, 76.2), turned to 180 degrees
- moved MX59 438.1 mm to (311.1, 95.2), turned to 180 degrees
- moved MX73 420.4 mm to (311.1, 114.3), turned to 180 degrees
- moved MX58 408.4 mm to (280.2, 95.2), turned to 180 degrees
- moved MX83 404.5 mm to (311.1, 133.3), turned to 180 degrees
- moved MX72 401.5 mm to (292.1, 114.3), turned to 180 degrees
- moved D16 392.0 mm to (315.9, 28.5), turned to -90 degrees
- moved MX82 387.0 mm to (292.1, 133.3), turned to 180 degrees
- moved D31 384.3 mm to (315.1, 52.3), turned to -90 degrees
- moved MX57 379.4 mm to (249.2, 95.2), turned to 180 degrees
- moved D46 377.2 mm to (314.3, 71.4), turned to -90 degrees
- moved MX71 376.1 mm to (265.9, 114.3), turned to 180 degrees
- moved D15 371.9 mm to (296.1, 28.6), turned to -90 degrees
- moved D60 371.9 mm to (315.1, 90.5), turned to -90 degrees
- moved MX81 370.3 mm to (273.1, 133.3), turned to 180 degrees
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Connections:
- D10 pad 1: col0 -> row0
- D11 pad 1: col0 -> row0
- D12 pad 1: col0 -> row0
- D13 pad 1: col0 -> row0
- D14 pad 1: col0 -> row0
- D15 pad 1: col0 -> row0
- D16 pad 1: col0 -> row0
- D17 pad 1: col0 -> row1
- D18 pad 1: col0 -> row1
- D19 pad 1: col0 -> row1
- D2 pad 1: col0 -> row0
- D20 pad 1: col0 -> row1
- D21 pad 1: col0 -> row1
- D22 pad 1: col0 -> row1
- D23 pad 1: col0 -> row1
- D24 pad 1: col0 -> row1
- D25 pad 1: col0 -> row1
- D26 pad 1: col0 -> row1
- D27 pad 1: col0 -> row1
- D28 pad 1: col0 -> row1
- D29 pad 1: col0 -> row1
- D3 pad 1: col0 -> row0
- D30 pad 1: col0 -> row1
- D31 pad 1: col0 -> row1
- D32 pad 1: col0 -> row2
- D33 pad 1: col0 -> row2
- D34 pad 1: col0 -> row2
- D35 pad 1: col0 -> row2
- D36 pad 1: col0 -> row2
- D37 pad 1: col0 -> row2
- D38 pad 1: col0 -> row2
- D39 pad 1: col0 -> row2
- D4 pad 1: col0 -> row0
- D40 pad 1: col0 -> row2
- D41 pad 1: col0 -> row2
- D42 pad 1: col0 -> row2
- D43 pad 1: col0 -> row2
- D44 pad 1: col0 -> row2
- D45 pad 1: col0 -> row2
- D46 pad 1: col0 -> row2
- D47 pad 1: col0 -> row3
- D48 pad 1: col0 -> row3
- D49 pad 1: col0 -> row3
- D5 pad 1: col0 -> row0
- D50 pad 1: col0 -> row3
- D51 pad 1: col0 -> row3
- D52 pad 1: col0 -> row3
- D53 pad 1: col0 -> row3
- D54 pad 1: col0 -> row3
- D55 pad 1: col0 -> row3
- D56 pad 1: col0 -> row3
- D57 pad 1: col0 -> row3
- D58 pad 1: col0 -> row3
- D59 pad 1: col0 -> row3
- D6 pad 1: col0 -> row0
- D60 pad 1: col0 -> row3
- D61 pad 1: col0 -> row4
- D62 pad 1: col0 -> row4
- D63 pad 1: col0 -> row4
- D64 pad 1: col0 -> row4
- D65 pad 1: col0 -> row4
- D66 pad 1: col0 -> row4
- D67 pad 1: col0 -> row4
- D68 pad 1: col0 -> row4
- D69 pad 1: col0 -> row4
- D7 pad 1: col0 -> row0
- D70 pad 1: col0 -> row4
- D71 pad 1: col0 -> row4
- D72 pad 1: col0 -> row4
- D73 pad 1: col0 -> row4
- D74 pad 1: col0 -> row4
- D75 pad 1: col0 -> row5
- D76 pad 1: col0 -> row5
- D77 pad 1: col0 -> row5
- D78 pad 1: col0 -> row5
- D79 pad 1: col0 -> row5
- D8 pad 1: col0 -> row0
- D80 pad 1: col0 -> row5
- D81 pad 1: col0 -> row5
- D82 pad 1: col0 -> row5
- D83 pad 1: col0 -> row5
- D84 pad 1: col0 -> row5
- D9 pad 1: col0 -> row0
- MX10 pad 2: col0 -> col9
- MX11 pad 2: col0 -> col10
- MX12 pad 2: col0 -> col11
- MX13 pad 2: col0 -> col12
- MX14 pad 2: col0 -> col13
- MX15 pad 2: col0 -> col14
- MX17 pad 2: col0 -> col1
- MX18 pad 2: col0 -> col2
- MX19 pad 2: col0 -> col3
- MX2 pad 2: col0 -> col1
- MX20 pad 2: col0 -> col4
- MX21 pad 2: col0 -> col5
- MX22 pad 2: col0 -> col6
- MX23 pad 2: col0 -> col7
- MX24 pad 2: col0 -> col8
- MX25 pad 2: col0 -> col9
- MX26 pad 2: col0 -> col10
- MX27 pad 2: col0 -> col11
- MX28 pad 2: col0 -> col12
- MX29 pad 2: col0 -> col13
- MX3 pad 2: col0 -> col2
- MX30 pad 2: col0 -> col14
- MX32 pad 2: col0 -> col1
- MX33 pad 2: col0 -> col2
- MX34 pad 2: col0 -> col3
- MX35 pad 2: col0 -> col4
- MX36 pad 2: col0 -> col5
- MX37 pad 2: col0 -> col6
- MX38 pad 2: col0 -> col7
- MX39 pad 2: col0 -> col8
- MX4 pad 2: col0 -> col3
- MX40 pad 2: col0 -> col9
- MX41 pad 2: col0 -> col10
- MX42 pad 2: col0 -> col11
- MX43 pad 2: col0 -> col12
- MX44 pad 2: col0 -> col13
- MX45 pad 2: col0 -> col14
- MX47 pad 2: col0 -> col1
- MX48 pad 2: col0 -> col2
- MX49 pad 2: col0 -> col4
- MX5 pad 2: col0 -> col4
- MX50 pad 2: col0 -> col5
- MX51 pad 2: col0 -> col6
- MX52 pad 2: col0 -> col7
- MX53 pad 2: col0 -> col8
- MX54 pad 2: col0 -> col9
- MX55 pad 2: col0 -> col10
- MX56 pad 2: col0 -> col11
- MX57 pad 2: col0 -> col12
- MX58 pad 2: col0 -> col13
- MX59 pad 2: col0 -> col14
- MX6 pad 2: col0 -> col5
- MX61 pad 2: col0 -> col1
- MX62 pad 2: col0 -> col2
- MX63 pad 2: col0 -> col4
- MX64 pad 2: col0 -> col5
- MX65 pad 2: col0 -> col6
- MX66 pad 2: col0 -> col7
- MX67 pad 2: col0 -> col8
- MX68 pad 2: col0 -> col9
- MX69 pad 2: col0 -> col10
- MX7 pad 2: col0 -> col6
- MX70 pad 2: col0 -> col11
- MX71 pad 2: col0 -> col12
- MX72 pad 2: col0 -> col13
- MX73 pad 2: col0 -> col14
- MX75 pad 2: col0 -> col1
- MX76 pad 2: col0 -> col2
- MX77 pad 2: col0 -> col6
- MX78 pad 2: col0 -> col9
- MX79 pad 2: col0 -> col10
- MX8 pad 2: col0 -> col7
- MX80 pad 2: col0 -> col11
- MX81 pad 2: col0 -> col12
- MX82 pad 2: col0 -> col13
- MX83 pad 2: col0 -> col14
- MX9 pad 2: col0 -> col8
- U1 pad 1: col0 -> row0
- U1 pad 11: col0 -> col14
- U1 pad 18: col0 -> col9
- U1 pad 19: col0 -> col10
- U1 pad 20: col0 -> col11
- U1 pad 21: col0 -> col12
- U1 pad 22: col0 -> col13
- U1 pad 25: col0 -> col8
- U1 pad 26: col0 -> col7
- U1 pad 27: col0 -> col6
- U1 pad 28: col0 -> col5
- U1 pad 30: col0 -> col1
- U1 pad 31: col0 -> col2
- U1 pad 32: col0 -> col3
- U1 pad 36: col0 -> col4
- U1 pad 37: col0 -> row5
- U1 pad 38: col0 -> row4
- U1 pad 39: col0 -> row3
- U1 pad 40: col0 -> row2
- U1 pad 41: col0 -> row1
Routing:
- net row1: track 0.00 -> 289.9 mm
- net row0: track 0.00 -> 288.3 mm, vias 0 -> 2
- net row3: track 0.00 -> 280.8 mm
- net row2: track 0.00 -> 280.3 mm
- net row4: track 0.00 -> 274.9 mm
- net row5: track 0.00 -> 213.1 mm
- net col12: track 0.00 -> 129.0 mm
- net col11: track 0.00 -> 126.7 mm
- net col10: track 0.00 -> 126.7 mm
- net col9: track 0.00 -> 126.4 mm
- net col1: track 0.00 -> 123.7 mm
- net col2: track 0.00 -> 120.5 mm
- net col13: track 0.00 -> 110.9 mm
- net col0: track 0.00 -> 108.3 mm
- net col7: track 0.00 -> 102.8 mm
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Other:
- board outline added: 308 x 127 mm
